Commit message: MoveIt fully integrated with tested planning and robot action. Changed planning to use TCP rather than link8. Partial scene planning implemented to avoid collision with environment.

File: src/pick_place_robot/urdf/panda.urdf (robot description, URDF)
Before this commit: robot panda, 14 links, 13 joints
Joints:
- joint panda_joint_base: origin xyz=0 0 0 rpy=0 0 0 -> xyz=0 0.6 0 rpy=0 0 -1.5708
