Commit message: added basic acquisition pipeline for simulated camera. added calibration mode to spawn robot with calibration target on tcp link for eye to hand calibration.

File: src/pick_place_robot/urdf/panda.urdf.xacro (robot description, xacro)
@@ -5,5 +5,6 @@
 <!-- =================================================================================== -->
 <!-- URDF for Franka Emika Panda -->
-<robot name="panda">
+<robot name="panda" xmlns:xacro="http://www.ros.org/wiki/xacro">
+  <xacro:arg name="enable_calibration" default="false"/>
   <link name="world">
   </link>
@@ -11,5 +12,5 @@
     <parent link="world"/>
     <child link="panda_link0"/>
-    <origin rpy="0 0 0" xyz="0 0 0"/>
+    <origin rpy="0 0 -1.5708" xyz="0 0.6 0"/>
   </joint>
   <link name="panda_link0">
@@ -17,11 +18,11 @@
       <origin rpy="0 0 0" xyz="0 0 0"/>
       <geometry>
-        <mesh filename="package://panda_description/meshes/visual/link0.dae"/>
-      </geometry>
-    </visual>
-    <collision>
-      <origin rpy="0 0 0" xyz="0 0 0"/>
-      <geometry>
-        <mesh filename="package://panda_description/meshes/collision/link0.stl"/>
+        <mesh filename="file:///home/michael/Projects/ROS2-PickAndPlaceRobot/install/panda_description/share/panda_description/meshes/visual/link0.dae"/>
+      </geometry>
+    </visual>
+    <collision>
+      <origin rpy="0 0 0" xyz="0 0 0"/>
+      <geometry>
+        <mesh filename="file:///home/michael/Projects/ROS2-PickAndPlaceRobot/install/panda_description/share/panda_description/meshes/collision/link0.stl"/>
       </geometry>
     </collision>
@@ -61,11 +62,11 @@
       <origin rpy="0 0 0" xyz="0 0 0"/>
       <geometry>
-        <mesh filename="package://panda_description/meshes/visual/link1.dae"/>
-      </geometry>
-    </visual>
-    <collision>
-      <origin rpy="0 0 0" xyz="0 0 0"/>
-      <geometry>
-        <mesh filename="package://panda_description/meshes/collision/link1.stl"/>
+        <mesh filename="file:///home/michael/Projects/ROS2-PickAndPlaceRobot/install/panda_description/share/panda_description/meshes/visual/link1.dae"/>
+      </geometry>
+    </visual>
+    <collision>
+      <origin rpy="0 0 0" xyz="0 0 0"/>
+      <geometry>
+        <mesh filename="file:///home/michael/Projects/ROS2-PickAndPlaceRobot/install/panda_description/share/panda_description/meshes/collision/link1.stl"/>
       </geometry>
     </collision>
@@ -105,11 +106,11 @@
       <origin rpy="0 0 0" xyz="0 0 0"/>
       <geometry>
-        <mesh filename="package://panda_description/meshes/visual/link2.dae"/>
-      </geometry>
-    </visual>
-    <collision>
-      <origin rpy="0 0 0" xyz="0 0 0"/>
-      <geometry>
-        <mesh filename="package://panda_description/meshes/collision/link2.stl"/>
+        <mesh filename="file:///home/michael/Projects/ROS2-PickAndPlaceRobot/install/panda_description/share/panda_description/meshes/visual/link2.dae"/>
+      </geometry>
+    </visual>
+    <collision>
+      <origin rpy="0 0 0" xyz="0 0 0"/>
+      <geometry>
+        <mesh filename="file:///home/michael/Projects/ROS2-PickAndPlaceRobot/install/panda_description/share/panda_description/meshes/collision/link2.stl"/>
       </geometry>
     </collision>
@@ -149,11 +150,11 @@
       <origin rpy="0 0 0" xyz="0 0 0"/>
       <geometry>
-        <mesh filename="package://panda_description/meshes/visual/link3.dae"/>
-      </geometry>
-    </visual>
-    <collision>
-      <origin rpy="0 0 0" xyz="0 0 0"/>
-      <geometry>
-        <mesh filename="package://panda_description/meshes/collision/link3.stl"/>
+        <mesh filename="file:///home/michael/Projects/ROS2-PickAndPlaceRobot/install/panda_description/share/panda_description/meshes/visual/link3.dae"/>
+      </geometry>
+    </visual>
+    <collision>
+      <origin rpy="0 0 0" xyz="0 0 0"/>
+      <geometry>
+        <mesh filename="file:///home/michael/Projects/ROS2-PickAndPlaceRobot/install/panda_description/share/panda_description/meshes/collision/link3.stl"/>
       </geometry>
     </collision>
@@ -193,11 +194,11 @@
       <origin rpy="0 0 0" xyz="0 0 0"/>
       <geometry>
-        <mesh filename="package://panda_description/meshes/visual/link4.dae"/>
-      </geometry>
-    </visual>
-    <collision>
-      <origin rpy="0 0 0" xyz="0 0 0"/>
-      <geometry>
-        <mesh filename="package://panda_description/meshes/collision/link4.stl"/>
+        <mesh filename="file:///home/michael/Projects/ROS2-PickAndPlaceRobot/install/panda_description/share/panda_description/meshes/visual/link4.dae"/>
+      </geometry>
+    </visual>
+    <collision>
+      <origin rpy="0 0 0" xyz="0 0 0"/>
+      <geometry>
+        <mesh filename="file:///home/michael/Projects/ROS2-PickAndPlaceRobot/install/panda_description/share/panda_description/meshes/collision/link4.stl"/>
       </geometry>
     </collision>
@@ -237,11 +238,11 @@
       <origin rpy="0 0 0" xyz="0 0 0"/>
       <geometry>
-        <mesh filename="package://panda_description/meshes/visual/link5.dae"/>
-      </geometry>
-    </visual>
-    <collision>
-      <origin rpy="0 0 0" xyz="0 0 0"/>
-      <geometry>
-        <mesh filename="package://panda_description/meshes/collision/link5.stl"/>
+        <mesh filename="file:///home/michael/Projects/ROS2-PickAndPlaceRobot/install/panda_description/share/panda_description/meshes/visual/link5.dae"/>
+      </geometry>
+    </visual>
+    <collision>
+      <origin rpy="0 0 0" xyz="0 0 0"/>
+      <geometry>
+        <mesh filename="file:///home/michael/Projects/ROS2-PickAndPlaceRobot/install/panda_description/share/panda_description/meshes/collision/link5.stl"/>
       </geometry>
     </collision>
@@ -281,11 +282,11 @@
       <origin rpy="0 0 0" xyz="0 0 0"/>
       <geometry>
-        <mesh filename="package://panda_description/meshes/visual/link6.dae"/>
-      </geometry>
-    </visual>
-    <collision>
-      <origin rpy="0 0 0" xyz="0 0 0"/>
-      <geometry>
-        <mesh filename="package://panda_description/meshes/collision/link6.stl"/>
+        <mesh filename="file:///home/michael/Projects/ROS2-PickAndPlaceRobot/install/panda_description/share/panda_description/meshes/visual/link6.dae"/>
+      </geometry>
+    </visual>
+    <collision>
+      <origin rpy="0 0 0" xyz="0 0 0"/>
+      <geometry>
+        <mesh filename="file:///home/michael/Projects/ROS2-PickAndPlaceRobot/install/panda_description/share/panda_description/meshes/collision/link6.stl"/>
       </geometry>
     </collision>
@@ -325,11 +326,11 @@
       <origin rpy="0 0 0" xyz="0 0 0"/>
       <geometry>
-        <mesh filename="package://panda_description/meshes/visual/link7.dae"/>
-      </geometry>
-    </visual>
-    <collision>
-      <origin rpy="0 0 0" xyz="0 0 0"/>
-      <geometry>
-        <mesh filename="package://panda_description/meshes/collision/link7.stl"/>
+        <mesh filename="file:///home/michael/Projects/ROS2-PickAndPlaceRobot/install/panda_description/share/panda_description/meshes/visual/link7.dae"/>
+      </geometry>
+    </visual>
+    <collision>
+      <origin rpy="0 0 0" xyz="0 0 0"/>
+      <geometry>
+        <mesh filename="file:///home/michael/Projects/ROS2-PickAndPlaceRobot/install/panda_description/share/panda_description/meshes/collision/link7.stl"/>
       </geometry>
     </collision>
@@ -414,11 +415,11 @@
       <origin rpy="0 0 0" xyz="0 0 0"/>
       <geometry>
-        <mesh filename="package://panda_description/meshes/visual/hand.dae"/>
-      </geometry>
-    </visual>
-    <collision>
-      <origin rpy="0 0 0" xyz="0 0 0"/>
-      <geometry>
-        <mesh filename="package://panda_description/meshes/collision/hand.stl"/>
+        <mesh filename="file:///home/michael/Projects/ROS2-PickAndPlaceRobot/install/panda_description/share/panda_description/meshes/visual/hand.dae"/>
+      </geometry>
+    </visual>
+    <collision>
+      <origin rpy="0 0 0" xyz="0 0 0"/>
+      <geometry>
+        <mesh filename="file:///home/michael/Projects/ROS2-PickAndPlaceRobot/install/panda_description/share/panda_description/meshes/collision/hand.stl"/>
       </geometry>
     </collision>
@@ -458,11 +459,11 @@
       <origin rpy="0 0 0" xyz="0 0 0"/>
       <geometry>
-        <mesh filename="package://panda_description/meshes/visual/finger.dae"/>
-      </geometry>
-    </visual>
-    <collision>
-      <origin rpy="0 0 0" xyz="0 0 0"/>
-      <geometry>
-        <mesh filename="package://panda_description/meshes/collision/finger.stl"/>
+        <mesh filename="file:///home/michael/Projects/ROS2-PickAndPlaceRobot/install/panda_description/share/panda_description/meshes/visual/finger.dae"/>
+      </geometry>
+    </visual>
+    <collision>
+      <origin rpy="0 0 0" xyz="0 0 0"/>
+      <geometry>
+        <mesh filename="file:///home/michael/Projects/ROS2-PickAndPlaceRobot/install/panda_description/share/panda_description/meshes/collision/finger.stl"/>
       </geometry>
     </collision>
@@ -502,5 +503,5 @@
       <origin rpy="0 0 3.141592653589793" xyz="0 0 0"/>
       <geometry>
-        <mesh filename="package://panda_description/meshes/visual/finger.dae"/>
+        <mesh filename="file:///home/michael/Projects/ROS2-PickAndPlaceRobot/install/panda_description/share/panda_description/meshes/visual/finger.dae"/>
       </geometry>
     </visual>
@@ -508,5 +509,5 @@
       <origin rpy="0 0 3.141592653589793" xyz="0 0 0"/>
       <geometry>
-        <mesh filename="package://panda_description/meshes/collision/finger.stl"/>
+        <mesh filename="file:///home/michael/Projects/ROS2-PickAndPlaceRobot/install/panda_description/share/panda_description/meshes/collision/finger.stl"/>
       </geometry>
     </collision>
@@ -528,4 +529,33 @@
     <origin rpy="0 0 0" xyz="0 0 0.1034"/>
   </joint>
+  <xacro:if value="$(arg enable_calibration)">
+    <link name="calibration_tag_link">
+      <visual>
+        <origin xyz="0 0 0" rpy="1.5708 0 0"/>
+        <geometry>
+          <mesh filename="file://$(find pick_place_robot)/meshes/april_tag_plate.dae"/>
+        </geometry>
+      </visual>
+      <collision>
+        <origin xyz="0 0 0" rpy="0 0 0"/>
+        <geometry>
+          <box size="0.08 0.01 0.08"/>
+        </geometry>
+      </collision>
+      <inertial>
+        <origin xyz="0 0 0" rpy="0 0 0"/>
+        <mass value="0.01"/>
+        <inertia ixx="0.00001" ixy="0.0" ixz="0.0" iyy="0.00001" iyz="0.0" izz="0.00001"/>
+      </inertial>
+    </link>
+    <joint name="calibration_tag_joint" type="fixed">
+      <parent link="panda_hand_tcp"/>
+      <child link="calibration_tag_link"/>
+      <origin xyz="0.0 0.0 0.010" rpy="0.0 0.0 0.0"/>
+    </joint>
+    <gazebo reference="calibration_tag_joint">
+      <preserveFixedJoint>true</preserveFixedJoint>
+    </gazebo>
+  </xacro:if>
   <ros2_control name="panda_gripper_system" type="system">
     <hardware>
