Commit message: Added tolerance checks and replanning after joint trajectories executed. Added homing recovery if the robot gets stuck in a position. Fixed image acquisition threads to prevent snapshot captures spinning and preventing sensor updates. Full calibration sequence and image capture completing correctly and consistantly.

File: src/pick_place_description/urdf/panda.urdf.xacro (robot description, xacro)
@@ -534,11 +534,13 @@
         <origin xyz="0 0 0" rpy="1.5708 0 0"/>
         <geometry>
-          <mesh filename="package://pick_place_description/meshes/april_tag_plate.dae"/>
+          <mesh
+            filename="package://pick_place_description/meshes/AprilTagBoard.obj"
+            scale="0.001 0.001 0.001"/>
         </geometry>
       </visual>
       <collision>
-        <origin xyz="0 0 0" rpy="0 0 0"/>
+        <origin xyz="0 0 0" rpy="1.5708 0 0"/>
         <geometry>
-          <box size="0.08 0.01 0.08"/>
+          <box size="0.25 0.005 0.25"/>
         </geometry>
       </collision>

Commit message: Implemented PDDL to handle operation sequence. Project working, improvements need implementing in future.

File: src/pick_place_description/urdf/panda.urdf.xacro (robot description, xacro)
@@ -439,5 +439,5 @@
     <origin rpy="0 0 0" xyz="0 0 0.0584"/>
     <axis xyz="0 1 0"/>
-    <limit effort="20" lower="0" upper="0.04" velocity="0.2"/>
+    <limit effort="40" lower="0" upper="0.04" velocity="0.2"/>
     <dynamics damping="3.0" friction="0.4"/>
   </joint>
@@ -483,5 +483,5 @@
     <origin rpy="0 0 0" xyz="0 0 0.0584"/>
     <axis xyz="0 -1 0"/>
-    <limit effort="20" lower="0" upper="0.04" velocity="0.2"/>
+    <limit effort="40" lower="0" upper="0.04" velocity="0.2"/>
     <dynamics damping="3.0" friction="0.4"/>
   </joint>
@@ -542,5 +542,5 @@
         <origin xyz="0 0 0" rpy="1.5708 0 0"/>
         <geometry>
-          <box size="0.25 0.005 0.25"/>
+          <box size="0.25 0.006 0.25"/>
         </geometry>
       </collision>
@@ -566,4 +566,22 @@
     <joint name="panda_finger_joint1">
       <param name="initial_position">0.0</param>
+      <!-- Explicit PID gains for ign_ros2_control's internal position
+           controller. Without these the plugin uses hardware defaults that
+           can be inconsistent between joints, causing one finger to respond
+           much faster than the other. Both joints use identical gains so
+           symmetric open/close motion is enforced.
+           kp=1000 matches the increased effort limit of 40 N: at full open
+           (0.04 m error) the PID outputs 1000 * 0.04 = 40 N, giving real
+           headroom above friction and gravity components at any wrist angle.
+           kd=30 targets critical damping: with finger mass ~0.224 kg the
+           undamped natural frequency is ωn = sqrt(kp/m) ≈ 67 rad/s, and
+           critical kd = 2·sqrt(kp·m) = 2·sqrt(1000·0.224) ≈ 30 N·s/m.
+           The previous kd=10 gave ζ ≈ 0.33 (underdamped), causing joint2
+           to overshoot onto the 0.040 m hard limit on short open moves
+           (e.g. 0.025 → 0.034 m after a grasp). kd=30 gives ζ ≈ 1.0
+           (critically damped), eliminating overshoot entirely. -->
+      <param name="kp">1000.0</param>
+      <param name="ki">0.0</param>
+      <param name="kd">30.0</param>
       <command_interface name="position"/>
       <state_interface name="position"/>
@@ -573,4 +591,7 @@
     <joint name="panda_finger_joint2">
       <param name="initial_position">0.0</param>
+      <param name="kp">1000.0</param>
+      <param name="ki">0.0</param>
+      <param name="kd">30.0</param>
       <command_interface name="position"/>
       <state_interface name="position"/>
